Commit message: Add files via upload

File: simulation/Maniskill/assets/fetch/fetch.urdf (robot description, URDF)
Before this commit: robot fetch, 30 links, 29 joints
Links:
- added link Left_Arm_Camera; visual mesh filename=meshes/XLeRobot_camera1.stl scale=0.001 0.001 0.001; visual mesh filename=meshes/XLeRobot_camera2.stl scale=0.001 0.001 0.001
- added link Right_Arm_Camera; visual mesh filename=meshes/XLeRobot_camera1.stl scale=0.001 0.001 0.001; visual mesh filename=meshes/XLeRobot_camera2.stl scale=0.001 0.001 0.001
- link base_link: geometry collision box size=0.009 0.405 0.09; collision box size=0.009 0.405 0.09
- link head_pan_link: geometry visual mesh filename=meshes/tophead3.stl scale=0.001 0.001 0.001; visual mesh filename=meshes/tophead4.stl scale=0.001 0.001 0.001
- link head_tilt_link: geometry visual mesh filename=meshes/tophead5.stl scale=0.001 0.001 0.001; visual mesh filename=meshes/tophead6.stl scale=0.001 0.001 0.001
- link top_base_link: geometry visual mesh filename=meshes/topbase1.stl scale=0.001 0.001 0.001; visual mesh filename=meshes/topbase2.stl scale=0.001 0.001 0.001
Joints:
- added joint Left_Arm_Camera_joint: type fixed, parent Fixed_Jaw_2, child Left_Arm_Camera, origin xyz=0 -0.02 -0.05 rpy=1.5708 0 -1.5708
- added joint Right_Arm_Camera_joint: type fixed, parent Fixed_Jaw, child Right_Arm_Camera, origin xyz=0 -0.02 -0.05 rpy=1.5708 0 -1.5708
- joint arm_base_joint: origin xyz=-0.14 -0.15 0.77 rpy=0 0 1.5708 -> xyz=-0.135 -0.133 0.760 rpy=0 0 1.5708
- joint arm_base_joint_2: origin xyz=-0.14 0.15 0.77 rpy=0 0 1.5708 -> xyz=-0.135 0.133 0.760 rpy=0 0 1.5708
- joint head_pan_joint: origin xyz=-0.125 0 0.18 rpy=0 0 0 -> xyz=-0.178 0 0 rpy=0 0 0
- joint head_tilt_joint: origin xyz=0.05 0 0.18 rpy=0 0 0 -> xyz=0.031 0 0.43815 rpy=0 0 0
- joint top_base_joint: origin xyz=0 0 0.73 rpy=-6.123E-17 0 0 -> xyz=0 0 0.73 rpy=0 0 0

Commit message: Add files via upload

File: simulation/Maniskill/assets/fetch/fetch.urdf (robot description, URDF)
Before this commit: robot fetch, 32 links, 31 joints
Joints:
- joint Left_Arm_Camera_joint: origin xyz=0 -0.02 -0.05 rpy=1.5708 0 -1.5708 -> xyz=0 -0.02 0.05 rpy=1.5708 0 -1.5708
- joint Right_Arm_Camera_joint: origin xyz=0 -0.02 -0.05 rpy=1.5708 0 -1.5708 -> xyz=0 -0.02 0.05 rpy=1.5708 0 -1.5708
