Commit message: xlerobot manskill simplification

File: simulation/Maniskill/assets/xlerobot/xlerobot.urdf (robot description, URDF)
Before this commit: robot xlerobot, 32 links, 31 joints
Joints:
- joint top_base_joint: origin xyz=0 0 0.73 rpy=0 0 0 -> xyz=0 0 0.73 rpy=0 0 3.14159

File: simulation/Maniskill/assets/xlerobot/xlerobot_front.urdf (robot description, URDF)
Before this commit: robot xlerobot_single, 22 links, 21 joints
Links:
- added link Base_2, mass 0.193184127927598; collision mesh filename=meshes/Base.stl; collision mesh filename=meshes/Base_Motor.stl
- added link Fixed_Jaw_2, mass 0.0929859131176897; collision mesh filename=meshes/Fixed_Jaw_part1.ply; collision mesh filename=meshes/Fixed_Jaw_part2.ply
- added link Fixed_Jaw_tip_2
- added link Left_Arm_Camera; visual mesh filename=meshes/XLeRobot_camera1.stl scale=0.001 0.001 0.001; visual mesh filename=meshes/XLeRobot_camera2.stl scale=0.001 0.001 0.001
- added link Lower_Arm_2, mass 0.147967774582291; collision mesh filename=meshes/Lower_Arm.stl; collision mesh filename=meshes/Lower_Arm_Motor.stl
- added link Moving_Jaw_2, mass 0.0202443794940372; collision mesh filename=meshes/Moving_Jaw_part1.ply; collision mesh filename=meshes/Moving_Jaw_part2.ply
- added link Moving_Jaw_tip_2
- added link Rotation_Pitch_2, mass 0.119226314127197; collision mesh filename=meshes/Rotation_Pitch.stl; collision mesh filename=meshes/Rotation_Pitch_Motor.stl
- added link Upper_Arm_2, mass 0.162409284599177; collision mesh filename=meshes/Upper_Arm.stl; collision mesh filename=meshes/Upper_Arm_Motor.stl
- added link Wrist_Pitch_Roll_2, mass 0.066132067097723; collision mesh filename=meshes/Wrist_Pitch_Roll.stl; collision mesh filename=meshes/Wrist_Pitch_Roll_Motor.stl
Joints:
- added joint Elbow_2: type revolute, parent Upper_Arm_2, child Lower_Arm_2, origin xyz=0 0.11257 0.028 rpy=-1.5708 0 0, axis 1 0 0, limit lower=-0.2 upper=3.14159 effort=0 velocity=0
- added joint Fixed_Jaw_tip_joint_2: type fixed, parent Fixed_Jaw_2, child Fixed_Jaw_tip_2, origin xyz=0.01 -0.097 0 rpy=0 0 0
- added joint Jaw_2: type revolute, parent Fixed_Jaw_2, child Moving_Jaw_2, origin xyz=-0.0202 -0.0244 0 rpy=3.1416 0 3.33, axis 0 0 1, limit lower=0 upper=1.7 effort=0 velocity=0
- added joint Left_Arm_Camera_joint: type fixed, parent Fixed_Jaw_2, child Left_Arm_Camera, origin xyz=0 -0.02 0.05 rpy=1.5708 0 -1.5708
- added joint Moving_Jaw_tip_joint_2: type fixed, parent Moving_Jaw_2, child Moving_Jaw_tip_2, origin xyz=-0.01 -0.073 0 rpy=0 0 0
- added joint Pitch_2: type revolute, parent Rotation_Pitch_2, child Upper_Arm_2, origin xyz=0 0.1025 0.0306 rpy=1.5708 0 0, axis -1 0 0, limit lower=-0.1 upper=3.45 effort=0 velocity=0
- added joint Rotation_2: type revolute, parent Base_2, child Rotation_Pitch_2, origin xyz=0 -0.0452 0.0165 rpy=1.5708 0 0, axis 0 -1 0, limit lower=-2.1 upper=2.1 effort=0 velocity=0
- added joint Wrist_Pitch_2: type revolute, parent Lower_Arm_2, child Wrist_Pitch_Roll_2, origin xyz=0 0.0052 0.1349 rpy=-1.5708 0 0, axis 1 0 0, limit lower=-1.8 upper=1.8 effort=0 velocity=0
- added joint Wrist_Roll_2: type revolute, parent Wrist_Pitch_Roll_2, child Fixed_Jaw_2, origin xyz=0 -0.0601 0 rpy=0 1.5708 0, axis 0 -1 0, limit lower=-3.14159 upper=3.14159 effort=0 velocity=0
- added joint arm_base_joint_2: type fixed, parent base_link, child Base_2, origin xyz=0.065 0.133 0.760 rpy=0 0 1.5708, axis 0 1 0, limit effort=8.85 velocity=17.4
- joint arm_base_joint: origin xyz=-0.135 -0.133 0.760 rpy=0 0 1.5708 -> xyz=0.065 -0.133 0.760 rpy=0 0 1.5708
- joint top_base_joint: origin xyz=0 0 0.73 rpy=0 0 0 -> xyz=0.2 0 0.73 rpy=0 0 0

Commit message: Fix top_base_joint

File: simulation/Maniskill/assets/xlerobot/xlerobot.urdf (robot description, URDF)
Before this commit: robot xlerobot, 32 links, 31 joints
Joints:
- joint top_base_joint: origin xyz=0 0 0.73 rpy=0 0 3.14159 -> xyz=0 0 0.73 rpy=0 0 0
